Commit message: Add RGB and depth cameras

File: install/robot_description/share/robot_description/urdf/robot.urdf (robot description, URDF)
Before this commit: robot my_robot, 5 links, 4 joints
Links:
- added link link_camera_optical_depth
- added link link_camera_optical_rgb
Joints:
- added joint joint_camera_optical_depth: type fixed, parent link_laser_scan, child link_camera_optical_depth, origin xyz=0 0 0 rpy=-1.570796 0 -1.570796
- added joint joint_camera_optical_rgb: type fixed, parent link_laser_scan, child link_camera_optical_rgb, origin xyz=0 0 0 rpy=-1.570796 0 -1.570796

File: install/robot_description/share/robot_description/urdf/robot.xacro (robot description, xacro)
@@ -180,4 +180,18 @@
             </collision>
         </link>
+        <!-- RGB Camera -->
+        <joint name="joint_camera_optical_rgb" type="fixed">
+            <origin rpy="-1.570796 0 -1.570796" xyz="0 0 0"/>
+            <parent link="link_laser_scan"/>
+            <child link="link_camera_optical_rgb"/>
+        </joint>
+        <link name="link_camera_optical_rgb"/>
+        <!-- Depth Camera -->
+        <joint name="joint_camera_optical_depth" type="fixed">
+            <origin rpy="-1.570796 0 -1.570796" xyz="0 0 0"/>
+            <parent link="link_laser_scan"/>
+            <child link="link_camera_optical_depth"/>
+        </joint>
+        <link name="link_camera_optical_depth"/>
     </robot>
 </xacro:root>
